File: Blink Eras.sch (KiCad schematic (older format))
At the start: 12 parts, among them IC1 ATTINY85-M, P1 ISP, U1 ICM7555

Commit message: Footprints, values, refinement.
Parts:
- C1: value C -> 1µ; footprint (none) -> Capacitors_SMD:C_0603_HandSoldering
- C2: value 100nF -> 1µ; footprint (none) -> Capacitors_SMD:C_0603_HandSoldering
- D1: value LED -> Red; footprint (none) -> LEDs:LED_0603
- D2: value LED -> Green; footprint (none) -> LEDs:LED_0603
- IC1: footprint QFN/MLF20 -> Housings_DFN_QFN:QFN-20-1EP_4x4mm_Pitch0.5mm
- R1: value R -> 1K
- R2: value R -> 470K
- R4: value R -> 56
- U1: footprint (none) -> Housings_SOIC:SOIC-8_3.9x4.9mm_Pitch1.27mm
Connections:
- net MOSI: no longer R4.1
- net at IC1.2 (PB3(XTAL1/CLKI/OC1B/ADC3/PCINT3)): now also R4.1
- net RESET renamed ~RESET~
- no-connect marks 3 -> 2
Other:
- moved on the sheet: C2, IC1, P1
Changed lines of the file:
@@
 L ATTINY85-M IC1
 U 1 1 577D47D3
-P 8050 3550
-F 0 "IC1" H 6900 3950 50  0000 C CNN
-F 1 "ATTINY85-M" H 9050 3150 50  0000 C CNN
-F 2 "QFN/MLF20" H 8900 3550 50  0000 C CIN
-F 3 "" H 8050 3550 50  0000 C CNN
-	1    8050 3550
+P 8050 3450
+F 0 "IC1" H 6900 3850 50  0000 C CNN
+F 1 "ATTINY85-M" H 9050 3050 50  0000 C CNN
+F 2 "Housings_DFN_QFN:QFN-20-1EP_4x4mm_Pitch0.5mm" H 8900 3450 50  0001 C CIN
+F 3 "" H 8050 3450 50  0000 C CNN
+	1    8050 3450
 	1    0    0    -1
 $EndComp
@@
 F 0 "BT1" H 5300 3500 50  0000 L CNN
 F 1 "Battery" H 5300 3400 50  0000 L CNN
-F 2 "" V 5200 3490 50  0000 C CNN
+F 2 "" V 5200 3490 50  0001 C CNN
 F 3 "" V 5200 3490 50  0000 C CNN
 	1    5200 3450
@@
 P 6100 3850
 F 0 "R4" V 6180 3850 50  0000 C CNN
-F 1 "R" V 6100 3850 50  0000 C CNN
-F 2 "" V 6030 3850 50  0000 C CNN
+F 1 "56" V 6100 3850 50  0000 C CNN
+F 2 "" V 6030 3850 50  0001 C CNN
 F 3 "" H 6100 3850 50  0000 C CNN
 	1    6100 3850
@@
 P 6100 4400
 F 0 "D2" H 6100 4500 50  0000 C CNN
-F 1 "LED" H 6100 4300 50  0000 C CNN
-F 2 "" H 6100 4400 50  0000 C CNN
+F 1 "Green" H 6100 4300 50  0000 C CNN
+F 2 "LEDs:LED_0603" H 6100 4400 50  0001 C CNN
 F 3 "" H 6100 4400 50  0000 C CNN
 	1    6100 4400
@@
 L CONN_02X03 P1
 U 1 1 577D50F2
-P 6950 2700
-F 0 "P1" H 6950 2900 50  0000 C CNN
-F 1 "ISP" H 6950 2500 50  0000 C CNN
-F 2 "" H 6950 1500 50  0000 C CNN
-F 3 "" H 6950 1500 50  0000 C CNN
-	1    6950 2700
-	1    0    0    -1
-$EndComp
+P 6950 2600
+F 0 "P1" H 6950 2800 50  0000 C CNN
+F 1 "ISP" H 6950 2400 50  0000 C CNN
+F 2 "" H 6950 1400 50  0001 C CNN
+F 3 "" H 6950 1400 50  0000 C CNN
+	1    6950 2600
+	1    0    0    -1
+$EndComp
+Text Label 6400 2500 0    60   ~ 0
+MISO
+Text Label 7500 2500 2    60   ~ 0
+VCC
+Text Label 7500 2600 2    60   ~ 0
+MOSI
+Text Label 7500 2700 2    60   ~ 0
+GND
 Text Label 6400 2600 0    60   ~ 0
+SCK
+Text Label 6400 2700 0    60   ~ 0
+~RESET~
+Text Label 6400 3200 0    60   ~ 0
+MOSI
+Text Label 6400 3300 0    60   ~ 0
 MISO
-Text Label 7500 2600 2    60   ~ 0
-VCC
-Text Label 7500 2700 2    60   ~ 0
-MOSI
-Text Label 7500 2800 2    60   ~ 0
-GND
-Text Label 6400 2700 0    60   ~ 0
+Text Label 6400 3400 0    60   ~ 0
 SCK
-Text Label 6400 2800 0    60   ~ 0
-RESET
-Text Label 6400 3300 0    60   ~ 0
-MOSI
-Text Label 6400 3400 0    60   ~ 0
-MISO
-Text Label 6400 3500 0    60   ~ 0
-SCK
-Text Label 6400 3800 0    60   ~ 0
-RESET
+Text Label 6400 3700 0    60   ~ 0
+~RESET~
 $Comp
 L R R1
@@
 P 2100 2950
 F 0 "R1" V 2180 2950 50  0000 C CNN
-F 1 "R" V 2100 2950 50  0000 C CNN
-F 2 "" V 2030 2950 50  0000 C CNN
+F 1 "1K" V 2100 2950 50  0000 C CNN
+F 2 "" V 2030 2950 50  0001 C CNN
 F 3 "" H 2100 2950 50  0000 C CNN
 	1    2100 2950
@@
 P 2100 3650
 F 0 "R2" V 2180 3650 50  0000 C CNN
-F 1 "R" V 2100 3650 50  0000 C CNN
-F 2 "" V 2030 3650 50  0000 C CNN
+F 1 "470K" V 2100 3650 50  0000 C CNN
+F 2 "" V 2030 3650 50  0001 C CNN
 F 3 "" H 2100 3650 50  0000 C CNN
 	1    2100 3650
@@
 P 2100 4350
 F 0 "C1" H 2125 4450 50  0000 L CNN
-F 1 "C" H 2125 4250 50  0000 L CNN
-F 2 "" H 2138 4200 50  0000 C CNN
+F 1 "1µ" H 2125 4250 50  0000 L CNN
+F 2 "Capacitors_SMD:C_0603_HandSoldering" H 2138 4200 50  0001 C CNN
 F 3 "" H 2100 4350 50  0000 C CNN
 	1    2100 4350
@@
 F 0 "R3" V 4380 3850 50  0000 C CNN
 F 1 "R" V 4300 3850 50  0000 C CNN
-F 2 "" V 4230 3850 50  0000 C CNN
+F 2 "" V 4230 3850 50  0001 C CNN
 F 3 "" H 4300 3850 50  0000 C CNN
 	1    4300 3850
@@
 L C C2
 U 1 1 577DCC0A
-P 9600 3550
-F 0 "C2" H 9625 3650 50  0000 L CNN
-F 1 "100nF" H 9625 3450 50  0000 L CNN
-F 2 "" H 9638 3400 50  0000 C CNN
-F 3 "" H 9600 3550 50  0000 C CNN
-	1    9600 3550
+P 9600 3450
+F 0 "C2" H 9625 3550 50  0000 L CNN
+F 1 "1µ" H 9625 3350 50  0000 L CNN
+F 2 "Capacitors_SMD:C_0603_HandSoldering" H 9638 3300 50  0001 C CNN
+F 3 "" H 9600 3450 50  0000 C CNN
+	1    9600 3450
 	1    0    0    -1
 $EndComp
@@
 P 4300 4400
 F 0 "D1" H 4300 4500 50  0000 C CNN
-F 1 "LED" H 4300 4300 50  0000 C CNN
-F 2 "" H 4300 4400 50  0000 C CNN
+F 1 "Red" H 4300 4300 50  0000 C CNN
+F 2 "LEDs:LED_0603" H 4300 4400 50  0001 C CNN
 F 3 "" H 4300 4400 50  0000 C CNN
 	1    4300 4400
@@
 F 0 "U1" H 2750 3950 60  0000 C CNN
 F 1 "ICM7555" H 3700 3050 60  0000 C CNN
-F 2 "" H 4100 3000 60  0000 C CNN
+F 2 "Housings_SOIC:SOIC-8_3.9x4.9mm_Pitch1.27mm" H 4100 3000 60  0001 C CNN
 F 3 "" H 4100 3000 60  0000 C CNN
 	1    3300 3500
@@
 $EndComp
 NoConn ~ 6700 3600
-NoConn ~ 6700 3700
 NoConn ~ 3400 4100
-Wire Wire Line
-	9400 3800 9600 3800
-Wire Wire Line
-	9400 3300 9600 3300
+Connection ~ 5200 3700
+Wire Wire Line
+	5500 3700 5500 3800
+Wire Wire Line
+	5200 3700 5500 3700
+Wire Wire Line
+	5200 3600 5200 5000
+Wire Wire Line
+	6100 4600 6100 5000
+Connection ~ 5200 3200
+Wire Wire Line
+	5500 3200 5200 3200
+Wire Wire Line
+	5500 3100 5500 3200
+Wire Wire Line
+	5200 2100 5200 3300
+Wire Wire Line
+	6100 4000 6100 4200
+Connection ~ 3400 2700
+Wire Wire Line
+	3200 2700 3400 2700
+Wire Wire Line
+	3400 2400 3400 2900
+Wire Wire Line
+	2100 2100 2100 2800
+Wire Wire Line
+	3200 2900 3200 2700
+Connection ~ 2100 2400
+Wire Wire Line
+	3400 2400 2100 2400
+Connection ~ 2400 3700
+Wire Wire Line
+	2500 3700 2400 3700
+Connection ~ 2100 4000
+Wire Wire Line
+	2400 4000 2100 4000
+Wire Wire Line
+	2400 3500 2400 4000
+Wire Wire Line
+	2500 3500 2400 3500
+Connection ~ 3200 4800
+Wire Wire Line
+	2100 4800 4300 4800
+Wire Wire Line
+	4300 4800 4300 4600
+Wire Wire Line
+	4300 4000 4300 4200
+Wire Wire Line
+	4300 3500 4100 3500
+Wire Wire Line
+	4300 3700 4300 3500
+Connection ~ 2100 4800
+Wire Wire Line
+	3200 4100 3200 4800
+Wire Wire Line
+	2100 4500 2100 5000
+Connection ~ 2100 3300
+Wire Wire Line
+	2500 3300 2100 3300
+Wire Wire Line
+	2100 3100 2100 3500
+Wire Wire Line
+	2100 3800 2100 4200
+Connection ~ 9600 3700
+Connection ~ 9600 3200
+Wire Wire Line
+	6400 3700 6700 3700
+Wire Wire Line
+	6400 3400 6700 3400
+Wire Wire Line
+	6400 3300 6700 3300
+Wire Wire Line
+	7200 2600 7500 2600
+Wire Wire Line
+	7200 2700 7500 2700
+Wire Wire Line
+	6400 2700 6700 2700
 Wire Wire Line
 	6400 2600 6700 2600
 Wire Wire Line
-	7200 2600 7500 2600
-Wire Wire Line
-	6400 2700 6700 2700
-Wire Wire Line
-	6400 2800 6700 2800
-Wire Wire Line
-	7200 2800 7500 2800
-Wire Wire Line
-	7200 2700 7500 2700
-Wire Wire Line
-	6400 3400 6700 3400
-Wire Wire Line
-	6400 3500 6700 3500
-Wire Wire Line
-	6400 3800 6700 3800
-Wire Wire Line
-	6700 3300 6100 3300
-Connection ~ 9600 3300
-Connection ~ 9600 3800
-Wire Wire Line
-	2100 4200 2100 3800
-Wire Wire Line
-	2100 3500 2100 3100
-Wire Wire Line
-	2500 3300 2100 3300
-Connection ~ 2100 3300
-Wire Wire Line
-	2100 4500 2100 5000
-Wire Wire Line
-	3200 4100 3200 4800
-Connection ~ 2100 4800
-Wire Wire Line
-	4300 3700 4300 3500
-Wire Wire Line
-	4300 3500 4100 3500
-Wire Wire Line
-	4300 4000 4300 4200
-Wire Wire Line
-	4300 4800 4300 4600
-Wire Wire Line
-	2100 4800 4300 4800
-Connection ~ 3200 4800
-Wire Wire Line
-	2500 3500 2400 3500
-Wire Wire Line
-	2400 3500 2400 4000
-Wire Wire Line
-	2400 4000 2100 4000
-Connection ~ 2100 4000
-Wire Wire Line
-	2500 3700 2400 3700
-Connection ~ 2400 3700
-Wire Wire Line
-	3400 2400 2100 2400
-Connection ~ 2100 2400
-Wire Wire Line
-	3200 2900 3200 2700
-Wire Wire Line
-	2100 2800 2100 2100
-Wire Wire Line
-	3400 2900 3400 2400
-Wire Wire Line
-	3200 2700 3400 2700
-Connection ~ 3400 2700
-Wire Wire Line
-	6100 3300 6100 3700
-Wire Wire Line
-	6100 4000 6100 4200
-Wire Wire Line
-	5200 3300 5200 2100
-Wire Wire Line
-	5500 3100 5500 3200
-Wire Wire Line
-	5500 3200 5200 3200
-Connection ~ 5200 3200
-Wire Wire Line
-	9600 2100 9600 3400
-Wire Wire Line
-	6100 4600 6100 5000
-Wire Wire Line
-	5200 3600 5200 5000
-Wire Wire Line
-	9600 3700 9600 5000
-Wire Wire Line
-	5200 3700 5500 3700
-Wire Wire Line
-	5500 3700 5500 3800
-Connection ~ 5200 3700
+	7200 2500 7500 2500
+Wire Wire Line
+	6400 2500 6700 2500
+Wire Wire Line
+	9400 3200 9600 3200
+Wire Wire Line
+	9400 3700 9600 3700
+Wire Wire Line
+	6700 3200 6400 3200
+Wire Wire Line
+	6700 3500 6100 3500
+Wire Wire Line
+	6100 3500 6100 3700
+Wire Wire Line
+	9600 2100 9600 3300
+Wire Wire Line
+	9600 3600 9600 5000
 $EndSCHEMATC
