File: KiCAD/Blink Eras.kicad_pcb (KiCad board)
At the start: 2 copper layers, 27.9 x 20.3 mm, 11 parts, among them IC1 ATTINY85-M, U1 ICM7555

Commit message: Battery holder was upside down.  Corrected.
Parts:
- turned BT1 to 180 degrees
Changed lines of the file:
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@@
   )
   (module BlinkyFeet:BK-913 (layer B.Cu)
-    (at 144.78 100.33)
-    (fp_text reference BT1 (at 0 -8.89) (layer B.SilkS) hide
+    (at 144.78 100.33 180)
+    (fp_text reference BT1 (at 0 -8.89 180) (layer B.SilkS) hide
       (effects (font (size 1 1) (thickness 0.15)) (justify mirror))
     )
-    (fp_text value CR2032 (at 0 7.62) (layer B.SilkS)
+    (fp_text value CR2032 (at 0 7.62 180) (layer B.SilkS)
       (effects (font (size 1 1) (thickness 0.15)) (justify mirror))
     )
     (fp_circle (center 0 0) (end 10 0) (layer B.SilkS) (width 0.15))
-    (pad 1 thru_hole circle (at -10.8 0) (size 4 4) (drill 2) (layers *.Cu *.Mask B.SilkS)
+    (pad 1 thru_hole circle (at -10.8 0 180) (size 4 4) (drill 2) (layers *.Cu *.Mask B.SilkS)
       (net 1 VCC))
-    (pad 2 smd rect (at 0 0) (size 3.96 3.96) (layers B.Cu B.Paste B.Mask)
+    (pad 2 smd rect (at 0 0 180) (size 3.96 3.96) (layers B.Cu B.Paste B.Mask)
       (net 2 GND))
-    (pad 1 thru_hole circle (at 10.8 0) (size 4 4) (drill 2) (layers *.Cu *.Mask B.SilkS)
+    (pad 1 thru_hole circle (at 10.8 0 180) (size 4 4) (drill 2) (layers *.Cu *.Mask B.SilkS)
       (net 1 VCC))
     (model "/Users/kbob/Documents/Making/Blink Eras/FreeCAD/BK-913.wrl"
