File: KiCAD/Blink Eras.sch (KiCad schematic (older format))
At the start: 12 parts, among them IC1 ATTINY85-M, P1 ISP, U1 ICM7555

Commit message: Added README and datasheets.
Parts:
- BT1: value Battery -> BK-913
- R1, R2, R4: footprint (none) -> Resistors_SMD:R_0603_HandSoldering
- R3: value R -> 68; footprint (none) -> Resistors_SMD:R_0603_HandSoldering
Changed lines of the file:
@@
 P 5200 3450
 F 0 "BT1" H 5300 3500 50  0000 L CNN
-F 1 "Battery" H 5300 3400 50  0000 L CNN
+F 1 "BK-913" H 5300 3400 50  0000 L CNN
 F 2 "" V 5200 3490 50  0001 C CNN
 F 3 "" V 5200 3490 50  0000 C CNN
@@
 F 0 "R4" V 6180 3850 50  0000 C CNN
 F 1 "56" V 6100 3850 50  0000 C CNN
-F 2 "" V 6030 3850 50  0001 C CNN
+F 2 "Resistors_SMD:R_0603_HandSoldering" V 6030 3850 50  0001 C CNN
 F 3 "" H 6100 3850 50  0000 C CNN
 	1    6100 3850
@@
 F 0 "R1" V 2180 2950 50  0000 C CNN
 F 1 "1K" V 2100 2950 50  0000 C CNN
-F 2 "" V 2030 2950 50  0001 C CNN
+F 2 "Resistors_SMD:R_0603_HandSoldering" V 2030 2950 50  0001 C CNN
 F 3 "" H 2100 2950 50  0000 C CNN
 	1    2100 2950
@@
 F 0 "R2" V 2180 3650 50  0000 C CNN
 F 1 "470K" V 2100 3650 50  0000 C CNN
-F 2 "" V 2030 3650 50  0001 C CNN
+F 2 "Resistors_SMD:R_0603_HandSoldering" V 2030 3650 50  0001 C CNN
 F 3 "" H 2100 3650 50  0000 C CNN
 	1    2100 3650
@@
 P 4300 3850
 F 0 "R3" V 4380 3850 50  0000 C CNN
-F 1 "R" V 4300 3850 50  0000 C CNN
-F 2 "" V 4230 3850 50  0001 C CNN
+F 1 "68" V 4300 3850 50  0000 C CNN
+F 2 "Resistors_SMD:R_0603_HandSoldering" V 4230 3850 50  0001 C CNN
 F 3 "" H 4300 3850 50  0000 C CNN
 	1    4300 3850

Commit message: Created footprint for BK-913 battery holder.
Parts:
- BT1: value BK-913 -> CR2032; footprint (none) -> BlinkyFeet:BK-913
Changed lines of the file:
@@
 P 5200 3450
 F 0 "BT1" H 5300 3500 50  0000 L CNN
-F 1 "BK-913" H 5300 3400 50  0000 L CNN
-F 2 "" V 5200 3490 50  0001 C CNN
+F 1 "CR2032" H 5300 3400 50  0000 L CNN
+F 2 "BlinkyFeet:BK-913" V 5200 3490 50  0001 C CNN
 F 3 "" V 5200 3490 50  0000 C CNN
 	1    5200 3450

Commit message: New layout makes the pogo pins fit.
Parts:
- P1: footprint (none) -> BlinkyFeet:ISP_Pogo_3-thru
Changed lines of the file:
@@
 F 0 "P1" H 6950 2800 50  0000 C CNN
 F 1 "ISP" H 6950 2400 50  0000 C CNN
-F 2 "" H 6950 1400 50  0001 C CNN
+F 2 "BlinkyFeet:ISP_Pogo_3-thru" H 6950 1400 50  0001 C CNN
 F 3 "" H 6950 1400 50  0000 C CNN
 	1    6950 2600

Commit message: Moved ATtiny bypass cap.
Parts:
- renumbered IC1 to U2
Changed lines of the file:
@@
 $EndDescr
 $Comp
-L ATTINY85-M IC1
+L ATTINY85-M U2
 U 1 1 577D47D3
 P 8050 3450
-F 0 "IC1" H 6900 3850 50  0000 C CNN
+F 0 "U2" H 6900 3850 50  0000 C CNN
 F 1 "ATTINY85-M" H 9050 3050 50  0000 C CNN
 F 2 "Housings_DFN_QFN:QFN-20-1EP_4x4mm_Pitch0.5mm" H 8900 3450 50  0001 C CIN
